Commit message: 修改左手為右手 	modified:   ex_ocare_control/config/controller_config.yaml 新增gmapping 和 laser_matcher功能 增加掃描LRF角度 	modified:   ex_ocare_control/launch/ocare_hw_node.xml 新增raspberry pi 端連線服務節點的launch檔 	new file:   ex_ocare_control/launch/ocare_network_daemon.launch 	new file:   ex_ocare_control/launch/ocare_network_daemon.xml 新增PC端控制與連線等相關節點的launch檔案 	new file:   ex_ocare_control/launch/ocare_pc_node.launch 	new file:   ex_ocare_control/launch/ocare_pc_node.xml 修改左手為右手（命名）並改善角度在robot_state_publisher的問題 	modified:   ex_ocare_control/src/ocare_hw_node.cpp 修正雷射測距儀的TF並增加了右手，並完成了TF設定 	modified:   labrob_description/urdf/ocare_realworld.urdf.xacro 新增語音控制介面和語音功能 	modified:   rqt_ocare/resource/ocare_ui.ui 	modified:   rqt_ocare/src/rqt_ocare/ocare_widget.py

File: labrob_description/urdf/ocare_realworld.urdf.xacro (robot description, xacro)
@@ -46,4 +46,31 @@
   <property name="left_arm_2_link_y_size" value="0.06" />
   <property name="left_arm_2_link_z_size" value="0.02" />
+    <!--Right Arm-base-->
+  <property name="right_arm_base_mass" value="0.20" />
+  <property name="right_arm_base_x_offset" value="0.0" />
+  <property name="right_arm_base_y_offset" value="0.0" />
+  <property name="right_arm_base_z_offset" value="-0.1" />
+  <property name="right_arm_base_x_size" value="0.05" />
+  <property name="right_arm_base_y_size" value="0.02" />
+  <property name="right_arm_base_z_size" value="0.10" />
+  <property name="base_x_origin_to_right_arm_base" value="0.0" />
+  <property name="base_y_origin_to_right_arm_base" value="-0.05" />
+  <property name="base_z_origin_to_right_arm_base" value="0.0" />
+    <!--Right Arm1-base-->
+  <property name="right_arm_1_link_mass" value="0.01" />
+  <property name="right_arm_1_link_x_offset" value="0.0" />
+  <property name="right_arm_1_link_y_offset" value="0.176" />
+  <property name="right_arm_1_link_z_offset" value="0.0" />
+  <property name="right_arm_1_link_x_size" value="0.05" />
+  <property name="right_arm_1_link_y_size" value="0.176" />
+  <property name="right_arm_1_link_z_size" value="0.02" />
+    <!--Right Arm2-base-->
+  <property name="right_arm_2_link_mass" value="0.01" />
+  <property name="right_arm_2_link_x_offset" value="-0.078" />
+  <property name="right_arm_2_link_y_offset" value="0.03" />
+  <property name="right_arm_2_link_z_offset" value="0.01" />
+  <property name="right_arm_2_link_x_size" value="0.078" />
+  <property name="right_arm_2_link_y_size" value="0.06" />
+  <property name="right_arm_2_link_z_size" value="0.02" />
 	<!--Camera Link-->
   <property name="camera_link_x_size" value="0.02" />
@@ -345,4 +372,172 @@
 	</joint>
 	<actuator name="left_arm_2_link_joint_actu">
+		<hardwareInterface>PositionJointInterface</hardwareInterface>
+		<mechanicalReduction>1</mechanicalReduction>
+	</actuator>
+  </transmission>
+  <!--Right-ARM-BASE-->
+  <link name="right_arm_base_link">
+    <inertial>
+      <mass value="${right_arm_base_mass}" />
+      <origin
+					xyz=
+				"${right_arm_base_x_offset} ${right_arm_base_y_offset} ${right_arm_base_z_offset-right_arm_base_z_size/2}"
+					rpy=
+				"0 0 0 " />
+      <!--The 3x3 rotational inertia matrix. -->
+       <box_inertia m="${right_arm_base_mass}" x="${right_arm_base_x_size}" y="${right_arm_base_y_size}" z="${right_arm_base_z_size}" />
+    </inertial>
+    <visual name="visual">
+      <origin
+					xyz=
+				"${right_arm_base_x_offset} ${right_arm_base_y_offset} ${right_arm_base_z_offset+right_arm_base_z_size/2}"
+					rpy=
+				"0 0 0 " />
+      <geometry>
+        <box size="${right_arm_base_x_size} ${right_arm_base_y_size} ${right_arm_base_z_size}" />
+      </geometry>
+      <material name="Green" />
+    </visual>
+	<collision>
+		<origin
+					xyz=
+				"${right_arm_base_x_offset-right_arm_base_x_size/2} ${right_arm_base_y_offset-right_arm_base_y_size/2} ${right_arm_base_z_offset-right_arm_base_z_size/2}"
+					rpy=
+				"0 0 0 " />
+      <geometry>
+        <box size="${right_arm_base_x_size} ${right_arm_base_y_size} ${right_arm_base_z_size}" />
+      </geometry>
+	</collision>
+  </link>
+  <gazebo reference="right_arm_base_link">
+    <material>Gazebo/Grey</material>
+    <turnGravityOff>false</turnGravityOff>
+  </gazebo>
+  <joint name="right_arm_base_link_joint" type="prismatic">
+	<parent link="base_link"/>
+	<child link="right_arm_base_link"/>
+	<origin xyz="${base_x_origin_to_right_arm_base} ${base_y_origin_to_right_arm_base} ${base_z_origin_to_right_arm_base}" rpy="${-M_PI/2} 0 0" />
+	<axis xyz="0 0 1"/>
+	<limit effort="100" velocity="100" lower="0" upper="0.15" />
+	<joint_properties damping="0.0" friction="0.0"/>
+  </joint>
+  <transmission name="right_arm_base_link_tran">
+	<type>transmission_interface/SimpleTransmission</type>
+	<joint name="right_arm_base_link_joint" >
+		<hardwareInterface>PositionJointInterface</hardwareInterface>
+	</joint>
+	<actuator name="right_arm_base_link_joint_actu">
+		<hardwareInterface>PositionJointInterface</hardwareInterface>
+		<mechanicalReduction>1</mechanicalReduction>
+	</actuator>
+  </transmission>
+   <!--RIGHT-ARM1-LINK-->
+  <link name="right_arm_1_link">
+    <inertial>
+      <mass value="${right_arm_1_link_mass}" />
+      <origin
+					xyz=
+				"${right_arm_1_link_x_offset} ${right_arm_1_link_y_offset-right_arm_1_link_y_size/2} ${right_arm_1_link_z_offset}"
+					rpy=
+				"0 0 0 " />
+      <!--The 3x3 rotational inertia matrix. -->
+       <box_inertia m="${right_arm_1_link_mass}" x="${right_arm_1_link_x_size}" y="${right_arm_1_link_y_size}" z="${right_arm_1_link_z_size}" />
+    </inertial>
+    <visual name="visual">
+      <origin
+					xyz=
+				"${right_arm_1_link_x_offset} ${right_arm_1_link_y_offset-right_arm_1_link_y_size/2} ${right_arm_1_link_z_offset}"
+					rpy=
+				"0 0 0 " />
+      <geometry>
+        <box size="${right_arm_1_link_x_size} ${right_arm_1_link_y_size} ${right_arm_1_link_z_size}" />
+      </geometry>
+      <material name="Green" />
+    </visual>
+	<collision>
+      <origin
+					xyz=
+				"${right_arm_1_link_x_offset} ${right_arm_1_link_y_offset-right_arm_1_link_y_size/2} ${right_arm_1_link_z_offset}"
+					rpy=
+				"0 0 0 " />
+      <geometry>
+        <box size="${right_arm_1_link_x_size} ${right_arm_1_link_y_size} ${right_arm_1_link_z_size}" />
+      </geometry>
+	</collision>
+  </link>
+  <gazebo reference="right_arm_1_link">
+    <material>Gazebo/Grey</material>
+    <turnGravityOff>false</turnGravityOff>
+  </gazebo>
+  <joint name="right_arm_1_link_joint" type="revolute">
+	<parent link="right_arm_base_link"/>
+	<child link="right_arm_1_link"/>
+	<origin xyz="${right_arm_base_x_offset} ${right_arm_base_y_offset} ${right_arm_base_z_offset}" rpy="0 0 0" />
+	<axis xyz="0 0 1"/>
+	<limit effort="5" velocity="1" lower="${-M_PI}" upper="0" />
+	<joint_properties damping="1.0" friction="0.0"/>
+  </joint>
+  <transmission name="right_arm_1_link_tran">
+  	<type>transmission_interface/SimpleTransmission</type>
+	<joint name="right_arm_1_link_joint" >
+		<hardwareInterface>PositionJointInterface</hardwareInterface>
+	</joint>
+	<actuator name="right_arm_1_link_joint_actu">
+		<hardwareInterface>PositionJointInterface</hardwareInterface>
+		<mechanicalReduction>1</mechanicalReduction>
+	</actuator>
+  </transmission>
+     <!--RIGHT-ARM2-LINK-->
+  <link name="right_arm_2_link">
+    <inertial>
+      <mass value="${right_arm_2_link_mass}" />
+      <origin
+					xyz=
+				"${right_arm_2_link_x_offset} ${right_arm_2_link_y_offset-right_arm_2_link_x_offset/2} ${right_arm_2_link_z_offset}"
+					rpy=
+				"0 0 0 " />
+      <!--The 3x3 rotational inertia matrix. -->
+       <box_inertia m="${right_arm_2_link_mass}" x="${right_arm_2_link_x_size}" y="${right_arm_2_link_y_size}" z="${right_arm_2_link_z_size}" />
+    </inertial>
+    <visual name="visual">
+      <origin
+					xyz=
+				"${right_arm_2_link_x_offset+right_arm_2_link_x_size/2} ${right_arm_2_link_y_offset} ${right_arm_2_link_z_offset}"
+					rpy=
+				"0 0 0 " />
+      <geometry>
+        <box size="${right_arm_2_link_x_size} ${right_arm_2_link_y_size} ${right_arm_2_link_z_size}" />
+      </geometry>
+      <material name="Red" />
+    </visual>
+	<collision>
+      <origin
+					xyz=
+				"${right_arm_2_link_x_offset+right_arm_2_link_x_size/2} ${right_arm_2_link_y_offset} ${right_arm_2_link_z_offset}"
+					rpy=
+				"0 0 0 " />
+      <geometry>
+        <box size="${right_arm_2_link_x_size} ${right_arm_2_link_y_size} ${right_arm_2_link_z_size}" />
+      </geometry>
+	</collision>
+  </link>
+  <gazebo reference="right_arm_2_link">
+    <material>Gazebo/Grey</material>
+    <turnGravityOff>false</turnGravityOff>
+  </gazebo>
+  <joint name="right_arm_2_link_joint" type="revolute">
+	<parent link="right_arm_1_link"/>
+	<child link="right_arm_2_link"/>
+	<origin xyz="${right_arm_1_link_x_offset} ${right_arm_1_link_y_offset} ${right_arm_1_link_z_offset}" rpy="0 0 ${M_PI/2}" />
+	<axis xyz="0 0 1"/>
+	<limit effort="5" velocity="1" lower="0" upper="${3*M_PI/2}" />
+	<joint_properties damping="1.0" friction="0.0"/>
+  </joint>
+  <transmission name="right_arm_2_link_tran">
+  	<type>transmission_interface/SimpleTransmission</type>
+	<joint name="right_arm_2_link_joint" >
+		<hardwareInterface>PositionJointInterface</hardwareInterface>
+	</joint>
+	<actuator name="right_arm_2_link_joint_actu">
 		<hardwareInterface>PositionJointInterface</hardwareInterface>
 		<mechanicalReduction>1</mechanicalReduction>
@@ -487,5 +682,5 @@
   <joint name="laser_joint" type="fixed">
     <axis xyz="0 1 0" />
-    <origin xyz="0 0 0" rpy="0 0 3.1416"/>
+    <origin xyz="0 0 0" rpy="0 0 0"/>
     <parent link="neck_link"/>
     <child link="laser"/>
